File: board/increment_button.kicad_pcb (KiCad board)
At the start: 2 copper layers, 5 parts, among them SW1 SW_Push_SPDT, U1 ER_OLEDM0.91_1x-I2C

Commit message: -
Parts:
- added D3: LED, LED_SMD:LED_01005_0402Metric, F.Cu at (156.9, 84.5)
- added R2: R, Resistor_THT:R_Axial_DIN0207_L6.3mm_D2.5mm_P10.16mm_Horizontal, F.Cu at (146.6, 73.5)
- added R3: R, Resistor_THT:R_Axial_DIN0207_L6.3mm_D2.5mm_P10.16mm_Horizontal, F.Cu at (146.6, 77.6)
- added R4: R, Resistor_THT:R_Axial_DIN0207_L6.3mm_D2.5mm_P10.16mm_Horizontal, F.Cu at (146.6, 81.6)
- added SW2: SW_Push_SPDT, Button_Switch_THT:SW_PUSH_6mm, F.Cu at (147.0, 85.7)
Connections:
- A1 pad 4: Net-(D1-K) -> Net-(D3-A)
- A1 pad 7: unconnected-(A1-D4-Pad7) -> Net-(A1-D4)
- R1 pad 2: Net-(A1-D2) -> Net-(A1-3V3)
- SW1 pad 2: Net-(A1-3V3) -> Net-(A1-D3)
- U1 pad 1: Net-(D1-K) -> Net-(D3-A)
Routing:
- net Net-(SW2-A): track 0.00 -> 13.2 mm
