File: board/increment_button.kicad_sch (KiCad schematic)
At the start: 0 parts

Commit message: added schematics and pcb
Parts:
- added A1: Arduino_Nano_v2.x, Module:Arduino_Nano, symbol MCU_Module:Arduino_Nano_v2.x
- added D1: LED, LED_THT:LED_D5.0mm, symbol Device:LED
- added R1: R, Resistor_THT:R_Axial_DIN0207_L6.3mm_D2.5mm_P10.16mm_Horizontal, symbol Device:R
- added SW1: SW_Push_SPDT, Button_Switch_THT:SW_PUSH_6mm, symbol Switch:SW_Push_SPDT
- added U1: ER_OLEDM0.91_1x-I2C, Display:ER_OLEDM0.91_1x-I2C, symbol Display_Graphic:ER_OLEDM0.91_1x-I2C
Connections:
- new net: R1.1, SW1.1 (A)
- new net: A1.17 (3V3), SW1.2 (B), U1.2 (VCC)
- new net: A1.6 (D3), SW1.3 (C)
- new net: A1.4 (GND), D1.1 (K), U1.1 (GND)
- new net: A1.24 (A5), U1.3 (SCL)
- new net: A1.23 (A4), U1.4 (SDA)
- new net: A1.5 (D2), D1.2 (A), R1.2

Commit message: changed sch
Parts:
- added D2: LED, symbol Device:LED
- added R2: R, Resistor_THT:R_Axial_DIN0207_L6.3mm_D2.5mm_P10.16mm_Horizontal, symbol Device:R
- added SW2: SW_Push_SPDT, Button_Switch_THT:SW_PUSH_6mm, symbol Switch:SW_Push_SPDT
- D1: footprint LED_THT:LED_D5.0mm -> (none)
Connections:
- net at A1.17 (3V3), U1.2 (VCC): now also D1.1 (K), R1.2, D2.1 (K), R2.2; no longer SW1.2 (B)
- net at A1.6 (D3): now also SW1.2 (B); no longer SW1.3 (C)
- net at A1.4 (GND), U1.1 (GND): now also SW1.3 (C), SW2.3 (C); no longer D1.1 (K)
- net at A1.5 (D2), D1.2 (A): no longer R1.2
- net at A1.7 (D4): now also SW2.2 (B)
- net at A1.8 (D5): now also D2.2 (A)
- new net: R2.1, SW2.1 (A)
- no-connect marks 0 -> 23
Other:
- moved on the sheet: R1, SW1

Commit message: -
Parts:
- added D3: LED, symbol Device:LED
- added R3, R4: R, Resistor_THT:R_Axial_DIN0207_L6.3mm_D2.5mm_P10.16mm_Horizontal, symbol Device:R
Connections:
- net at A1.4 (GND), SW1.3 (C), SW2.3 (C)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: now also D3.1 (K), D3.2 (A)
- net at D1.2 (A): now also R3.2; no longer A1.5 (D2)
- net at D2.2 (A): now also R4.2; no longer A1.8 (D5)
- new net: A1.5 (D2), R3.1
- new net: A1.8 (D5), R4.1
Other:
- moved on the sheet: D2

Commit message: -
Parts:
- removed D3: LED, symbol Device:LED
Changed lines of the file:
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@@
-	)
-	(junction
-		(at 176.53 106.68)
-		(diameter 0)
-		(color 0 0 0 0)
 	)
 	(junction
@@
 		(color 0 0 0 0)
 	)
-	(junction
-		(at 176.53 97.79)
-		(diameter 0)
-		(color 0 0 0 0)
-	)
 	(no_connect
 		(at 90.17 73.66)
@@
 	(wire
 		(pts
-			(xy 191.77 97.79) (xy 176.53 97.79)
-		)
-		(stroke
-			(width 0)
-			(type default)
-		)
-	)
-	(wire
-		(pts
 			(xy 176.53 67.31) (xy 179.07 67.31)
 		)
@@
 	(wire
 		(pts
-			(xy 176.53 97.79) (xy 176.53 106.68)
-		)
-		(stroke
-			(width 0)
-			(type default)
-		)
-	)
-	(wire
-		(pts
 			(xy 176.53 76.2) (xy 201.93 76.2)
 		)
@@
 	(wire
 		(pts
-			(xy 191.77 106.68) (xy 191.77 105.41)
-		)
-		(stroke
-			(width 0)
-			(type default)
-		)
-	)
-	(wire
-		(pts
 			(xy 62.23 48.26) (xy 62.23 78.74)
 		)
@@
 	(wire
 		(pts
-			(xy 176.53 106.68) (xy 191.77 106.68)
-		)
-		(stroke
-			(width 0)
-			(type default)
-		)
-	)
-	(wire
-		(pts
 			(xy 80.01 53.34) (xy 128.27 53.34)
 		)
@@
 	(wire
 		(pts
-			(xy 176.53 76.2) (xy 176.53 97.79)
-		)
-		(stroke
-			(width 0)
-			(type default)
-		)
-	)
-	(wire
-		(pts
 			(xy 49.53 36.83) (xy 49.53 83.82)
 		)
@@
 	(wire
 		(pts
+			(xy 176.53 76.2) (xy 176.53 127)
+		)
+		(stroke
+			(width 0)
+			(type default)
+		)
+	)
+	(wire
+		(pts
 			(xy 212.09 53.34) (xy 212.09 67.31)
 		)
@@
 		(pts
 			(xy 190.5 69.85) (xy 190.5 36.83)
-		)
-		(stroke
-			(width 0)
-			(type default)
-		)
-	)
-	(wire
-		(pts
-			(xy 176.53 127) (xy 176.53 106.68)
 		)
 		(stroke
@@
 					(unit 1)
 				)
-			)
-		)
-	)
-	(symbol
-		(lib_id "Device:LED")
-		(at 191.77 101.6 270)
-		(unit 1)
-		(body_style 1)
-		(exclude_from_sim no)
-		(in_bom yes)
-		(on_board yes)
-		(in_pos_files yes)
-		(dnp no)
-		(fields_autoplaced yes)
-		(property "Reference" "D3"
-			(at 194.31 98.7424 90)
-			(show_name no)
-			(do_not_autoplace no)
-			(effects
-				(font
-					(size 1.27 1.27)
-				)
-				(justify left)
-			)
-		)
-		(property "Value" "LED"
-			(at 194.31 101.2824 90)
-			(show_name no)
-			(do_not_autoplace no)
-			(effects
-				(font
-					(size 1.27 1.27)
-				)
-				(justify left)
-			)
-		)
-		(property "Footprint" ""
-			(at 191.77 101.6 0)
-			(hide yes)
-			(show_name no)
-			(do_not_autoplace no)
-			(effects
-				(font
-					(size 1.27 1.27)
-				)
-			)
-		)
-		(property "Datasheet" ""
-			(at 191.77 101.6 0)
-			(hide yes)
-			(show_name no)
-			(do_not_autoplace no)
-			(effects
-				(font
-					(size 1.27 1.27)
-				)
-			)
-		)
-		(property "Description" "Light emitting diode"
-			(at 191.77 101.6 0)
-			(hide yes)
-			(show_name no)
-			(do_not_autoplace no)
-			(effects
-				(font
-					(size 1.27 1.27)
-				)
-			)
-		)
-		(property "Sim.Pins" "1=K 2=A"
-			(at 191.77 101.6 0)
-			(hide yes)
-			(show_name no)
-			(do_not_autoplace no)
-			(effects
-				(font
-					(size 1.27 1.27)
-				)
-			)
-		)
-		(pin "1"
-		)
-		(pin "2"
-		)
-		(instances
-			(project "increment_button"
-				(path "/7090d103-b608-433c-8c6c-b1ecb5c61ded"
-					(reference "D3")
-					(unit 1)
-				)

Commit message: -
Parts:
- added D3: LED, LED_SMD:LED_01005_0402Metric, symbol Device:LED
Connections:
- net at A1.4 (GND), SW1.3 (C), SW2.3 (C)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: now also D3.1 (K), D3.2 (A)
Changed lines of the file:
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@@
 	(paper "A4")
+	(junction
+		(at 176.53 95.25)
+		(diameter 0)
+		(color 0 0 0 0)
+	)
 	(junction
 		(at 176.53 76.2)
@@
 		(color 0 0 0 0)
 	)
+	(junction
+		(at 176.53 102.87)
+		(diameter 0)
+		(color 0 0 0 0)
+	)
 	(no_connect
 		(at 90.17 73.66)
@@
 	(wire
 		(pts
+			(xy 176.53 102.87) (xy 186.69 102.87)
+		)
+		(stroke
+			(width 0)
+			(type default)
+		)
+	)
+	(wire
+		(pts
 			(xy 60.96 86.36) (xy 60.96 50.8)
 		)
@@
 	(wire
 		(pts
+			(xy 176.53 95.25) (xy 186.69 95.25)
+		)
+		(stroke
+			(width 0)
+			(type default)
+		)
+	)
+	(wire
+		(pts
 			(xy 62.23 48.26) (xy 62.23 78.74)
 		)
@@
 	(wire
 		(pts
+			(xy 176.53 102.87) (xy 176.53 127)
+		)
+		(stroke
+			(width 0)
+			(type default)
+		)
+	)
+	(wire
+		(pts
 			(xy 80.01 53.34) (xy 128.27 53.34)
 		)
@@
 	(wire
 		(pts
+			(xy 176.53 95.25) (xy 176.53 102.87)
+		)
+		(stroke
+			(width 0)
+			(type default)
+		)
+	)
+	(wire
+		(pts
 			(xy 49.53 36.83) (xy 49.53 83.82)
 		)
@@
 	(wire
 		(pts
-			(xy 176.53 76.2) (xy 176.53 127)
+			(xy 176.53 76.2) (xy 176.53 95.25)
 		)
 		(stroke
@@
 					(unit 1)
 				)
+			)
+		)
+	)
+	(symbol
+		(lib_id "Device:LED")
+		(at 186.69 99.06 90)
+		(unit 1)
+		(body_style 1)
+		(exclude_from_sim no)
+		(in_bom yes)
+		(on_board yes)
+		(in_pos_files yes)
+		(dnp no)
+		(fields_autoplaced yes)
+		(property "Reference" "D3"
+			(at 190.5 99.3774 90)
+			(show_name no)
+			(do_not_autoplace no)
+			(effects
+				(font
+					(size 1.27 1.27)
+				)
+				(justify right)
+			)
+		)
+		(property "Value" "LED"
+			(at 190.5 101.9174 90)
+			(show_name no)
+			(do_not_autoplace no)
+			(effects
+				(font
+					(size 1.27 1.27)
+				)
+				(justify right)
+			)
+		)
+		(property "Footprint" "LED_SMD:LED_01005_0402Metric"
+			(at 186.69 99.06 0)
+			(hide yes)
+			(show_name no)
+			(do_not_autoplace no)
+			(effects
+				(font
+					(size 1.27 1.27)
+				)
+			)
+		)
+		(property "Datasheet" ""
+			(at 186.69 99.06 0)
+			(hide yes)
+			(show_name no)
+			(do_not_autoplace no)
+			(effects
+				(font
+					(size 1.27 1.27)
+				)
+			)
+		)
+		(property "Description" "Light emitting diode"
+			(at 186.69 99.06 0)
+			(hide yes)
+			(show_name no)
+			(do_not_autoplace no)
+			(effects
+				(font
+					(size 1.27 1.27)
+				)
+			)
+		)
+		(property "Sim.Pins" "1=K 2=A"
+			(at 186.69 99.06 0)
+			(hide yes)
+			(show_name no)
+			(do_not_autoplace no)
+			(effects
+				(font
+					(size 1.27 1.27)
+				)
+			)
+		)
+		(pin "2"
+		)
+		(pin "1"
+		)
+		(instances
+			(project "increment_button"
+				(path "/7090d103-b608-433c-8c6c-b1ecb5c61ded"
+					(reference "D3")
+					(unit 1)
+				)
